File: pcb/pcb.kicad_pcb (KiCad board)
At the start: 2 copper layers, 124 parts, among them J1 AVR-ISP-6, SW1 BOOT, SW2 RESET, U1 ATmega328P-P, Y1 Crystal

Commit message: 🚧 Fixing diodes footprints issue
Parts:
- removed REF** (x2): Stabilizer_Cherry_MX_2.00u, Mounting_Keyboard_Stabilizer:Stabilizer_Cherry_MX_2.00u
- moved D37 200.5 mm to (44.5, 54.9), turned to -90 degrees
- moved D26 197.7 mm to (54.0, 54.9), turned to -90 degrees
- moved D13 192.1 mm to (38.1, 54.9), turned to -90 degrees
- moved D27 189.3 mm to (66.7, 54.9), turned to -90 degrees
- moved D12 185.7 mm to (259.6, 55.7), turned to -90 degrees
- moved D38 181.7 mm to (57.1, 54.9), turned to -90 degrees
- moved D41 176.0 mm to (95.2, 54.9), turned to -90 degrees
- moved D48 175.5 mm to (269.1, 55.7), turned to -90 degrees
- moved D39 174.1 mm to (69.8, 54.9), turned to -90 degrees
- moved D44 172.0 mm to (218.3, 55.7), turned to -90 degrees
- moved D28 171.9 mm to (79.4, 54.9), turned to -90 degrees
- moved D34 170.4 mm to (240.5, 55.7), turned to -90 degrees
- moved D4 169.6 mm to (73.0, 54.9), turned to -90 degrees
- moved D25 166.7 mm to (41.3, 54.9), turned to -90 degrees
- moved D18 166.5 mm to (101.6, 54.9), turned to -90 degrees
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Connections:
- D1 pad 1: Net-(D1-Pad1) -> row0
- D1 pad 2: row0 -> Net-(D1-Pad2)
- D10 pad 1: Net-(D10-Pad1) -> row0
- D10 pad 2: row0 -> Net-(D10-Pad2)
- D11 pad 1: Net-(D11-Pad1) -> row0
- D11 pad 2: row0 -> Net-(D11-Pad2)
- D12 pad 1: Net-(D12-Pad1) -> row0
- D12 pad 2: row0 -> Net-(D12-Pad2)
- D13 pad 1: Net-(D13-Pad1) -> row1
- D13 pad 2: row1 -> Net-(D13-Pad2)
- D14 pad 1: Net-(D14-Pad1) -> row1
- D14 pad 2: row1 -> Net-(D14-Pad2)
- D15 pad 1: Net-(D15-Pad1) -> row1
- D15 pad 2: row1 -> Net-(D15-Pad2)
- D16 pad 1: Net-(D16-Pad1) -> row1
- D16 pad 2: row1 -> Net-(D16-Pad2)
- D17 pad 1: Net-(D17-Pad1) -> row1
- D17 pad 2: row1 -> Net-(D17-Pad2)
- D18 pad 1: Net-(D18-Pad1) -> row1
- D18 pad 2: row1 -> Net-(D18-Pad2)
- D19 pad 1: Net-(D19-Pad1) -> row1
- D19 pad 2: row1 -> Net-(D19-Pad2)
- D2 pad 1: Net-(D2-Pad1) -> row0
- D2 pad 2: row0 -> Net-(D2-Pad2)
- D20 pad 1: Net-(D20-Pad1) -> row1
- D20 pad 2: row1 -> Net-(D20-Pad2)
- D21 pad 1: Net-(D21-Pad1) -> row1
- D21 pad 2: row1 -> Net-(D21-Pad2)
- D22 pad 1: Net-(D22-Pad1) -> row1
- D22 pad 2: row1 -> Net-(D22-Pad2)
- D23 pad 1: Net-(D23-Pad1) -> row1
- D23 pad 2: row1 -> Net-(D23-Pad2)
- D24 pad 1: Net-(D24-Pad1) -> row1
- D24 pad 2: row1 -> Net-(D24-Pad2)
- D25 pad 1: Net-(D25-Pad1) -> row2
- D25 pad 2: row2 -> Net-(D25-Pad2)
- D26 pad 1: Net-(D26-Pad1) -> row2
- D26 pad 2: row2 -> Net-(D26-Pad2)
- D27 pad 1: Net-(D27-Pad1) -> row2
- D27 pad 2: row2 -> Net-(D27-Pad2)
- D28 pad 1: Net-(D28-Pad1) -> row2
- D28 pad 2: row2 -> Net-(D28-Pad2)
- D29 pad 1: Net-(D29-Pad1) -> row2
- D29 pad 2: row2 -> Net-(D29-Pad2)
- D3 pad 1: Net-(D3-Pad1) -> row0
- D3 pad 2: row0 -> Net-(D3-Pad2)
- D30 pad 1: Net-(D30-Pad1) -> row2
- D30 pad 2: row2 -> Net-(D30-Pad2)
- D31 pad 1: Net-(D31-Pad1) -> row2
- D31 pad 2: row2 -> Net-(D31-Pad2)
- D32 pad 1: Net-(D32-Pad1) -> row2
- D32 pad 2: row2 -> Net-(D32-Pad2)
- D33 pad 1: Net-(D33-Pad1) -> row2
- D33 pad 2: row2 -> Net-(D33-Pad2)
- D34 pad 1: Net-(D34-Pad1) -> row2
- D34 pad 2: row2 -> Net-(D34-Pad2)
- D35 pad 1: Net-(D35-Pad1) -> row2
- D35 pad 2: row2 -> Net-(D35-Pad2)
- D36 pad 1: Net-(D36-Pad1) -> row2
- D36 pad 2: row2 -> Net-(D36-Pad2)
- D37 pad 1: Net-(D37-Pad1) -> col1
- D37 pad 2: col1 -> Net-(S37-Pad2)
- D38 pad 1: Net-(D38-Pad1) -> col1
- D38 pad 2: col1 -> Net-(D38-Pad2)
- D39 pad 1: Net-(D39-Pad1) -> col1
- D39 pad 2: col1 -> Net-(D39-Pad2)
- D4 pad 1: Net-(D4-Pad1) -> row0
- D4 pad 2: row0 -> Net-(D4-Pad2)
- D40 pad 1: Net-(D40-Pad1) -> col1
- D40 pad 2: col1 -> Net-(D40-Pad2)
- D41 pad 1: Net-(D41-Pad1) -> col1
- D41 pad 2: col1 -> Net-(D41-Pad2)
- D42 pad 1: unconnected-(D42-Pad1) -> col1
- D42 pad 2: col1 -> unconnected-(D42-Pad2)
- D43 pad 1: Net-(D43-Pad1) -> col1
- D43 pad 2: col1 -> Net-(D43-Pad2)
- D44 pad 1: unconnected-(D44-Pad1) -> col1
- D44 pad 2: col1 -> unconnected-(D44-Pad2)
- D45 pad 1: Net-(D45-Pad1) -> col1
- D45 pad 2: col1 -> Net-(D45-Pad2)
- D46 pad 1: Net-(D46-Pad1) -> col1
- D46 pad 2: col1 -> Net-(D46-Pad2)
- D47 pad 1: Net-(D47-Pad1) -> col1
- D47 pad 2: col1 -> Net-(D47-Pad2)
- D48 pad 1: Net-(D48-Pad1) -> col1
- D48 pad 2: col1 -> Net-(D48-Pad2)
- D5 pad 1: Net-(D5-Pad1) -> row0
- D5 pad 2: row0 -> Net-(D5-Pad2)
- D6 pad 1: Net-(D6-Pad1) -> row0
- D6 pad 2: row0 -> Net-(D6-Pad2)
- D7 pad 1: Net-(D7-Pad1) -> row0
- D7 pad 2: row0 -> Net-(D7-Pad2)
- D8 pad 1: Net-(D8-Pad1) -> row0
- D8 pad 2: row0 -> Net-(D8-Pad2)
- D9 pad 1: Net-(D9-Pad1) -> row0
- D9 pad 2: row0 -> Net-(D9-Pad2)
- S1 pad 2: Net-(D1-Pad1) -> Net-(D1-Pad2)
- S10 pad 2: Net-(D10-Pad1) -> Net-(D10-Pad2)
- S11 pad 2: Net-(D11-Pad1) -> Net-(D11-Pad2)
- S12 pad 2: Net-(D12-Pad1) -> Net-(D12-Pad2)
- S13 pad 2: Net-(D13-Pad1) -> Net-(D13-Pad2)
- S14 pad 2: Net-(D14-Pad1) -> Net-(D14-Pad2)
- S15 pad 2: Net-(D15-Pad1) -> Net-(D15-Pad2)
- S16 pad 2: Net-(D16-Pad1) -> Net-(D16-Pad2)
- S17 pad 2: Net-(D17-Pad1) -> Net-(D17-Pad2)
- S18 pad 2: Net-(D18-Pad1) -> Net-(D18-Pad2)
- S19 pad 2: Net-(D19-Pad1) -> Net-(D19-Pad2)
- S2 pad 2: Net-(D2-Pad1) -> Net-(D2-Pad2)
- S20 pad 2: Net-(D20-Pad1) -> Net-(D20-Pad2)
- S21 pad 2: Net-(D21-Pad1) -> Net-(D21-Pad2)
- S22 pad 2: Net-(D22-Pad1) -> Net-(D22-Pad2)
- S23 pad 2: Net-(D23-Pad1) -> Net-(D23-Pad2)
- S24 pad 2: Net-(D24-Pad1) -> Net-(D24-Pad2)
- S25 pad 2: Net-(D25-Pad1) -> Net-(D25-Pad2)
- S26 pad 2: Net-(D26-Pad1) -> Net-(D26-Pad2)
- S27 pad 2: Net-(D27-Pad1) -> Net-(D27-Pad2)
- S28 pad 2: Net-(D28-Pad1) -> Net-(D28-Pad2)
- S29 pad 2: Net-(D29-Pad1) -> Net-(D29-Pad2)
- S3 pad 2: Net-(D3-Pad1) -> Net-(D3-Pad2)
- S30 pad 2: Net-(D30-Pad1) -> Net-(D30-Pad2)
- S31 pad 2: Net-(D31-Pad1) -> Net-(D31-Pad2)
- S32 pad 2: Net-(D32-Pad1) -> Net-(D32-Pad2)
- S33 pad 2: Net-(D33-Pad1) -> Net-(D33-Pad2)
- S34 pad 2: Net-(D34-Pad1) -> Net-(D34-Pad2)
- S35 pad 2: Net-(D35-Pad1) -> Net-(D35-Pad2)
- S36 pad 2: Net-(D36-Pad1) -> Net-(D36-Pad2)
- S37 pad 2: Net-(D37-Pad1) -> Net-(S37-Pad2)
- S38 pad 2: Net-(D38-Pad1) -> Net-(D38-Pad2)
- S39 pad 1: col2 -> col3
- S39 pad 2: Net-(D39-Pad1) -> Net-(D40-Pad2)
- S4 pad 2: Net-(D4-Pad1) -> Net-(D4-Pad2)
- S40 pad 2: Net-(D41-Pad1) -> Net-(D41-Pad2)
- S41 pad 2: Net-(D43-Pad1) -> Net-(D43-Pad2)
- S42 pad 2: Net-(D45-Pad1) -> Net-(D45-Pad2)
- S43 pad 2: Net-(D46-Pad1) -> Net-(D46-Pad2)
- S44 pad 2: Net-(D48-Pad1) -> Net-(D48-Pad2)
- S45 pad 2: Net-(D37-Pad1) -> Net-(S37-Pad2)
- S46 pad 2: Net-(D38-Pad1) -> Net-(D38-Pad2)
- S47 pad 2: Net-(D39-Pad1) -> Net-(D39-Pad2)
- S48 pad 2: Net-(D40-Pad1) -> Net-(D40-Pad2)
- S49 pad 2: Net-(D45-Pad1) -> Net-(D45-Pad2)
- S5 pad 2: Net-(D5-Pad1) -> Net-(D5-Pad2)
- S50 pad 2: Net-(D46-Pad1) -> Net-(D46-Pad2)
- S51 pad 2: Net-(D47-Pad1) -> Net-(D47-Pad2)
- S52 pad 2: Net-(D48-Pad1) -> Net-(D48-Pad2)
- S6 pad 2: Net-(D6-Pad1) -> Net-(D6-Pad2)
- S7 pad 2: Net-(D7-Pad1) -> Net-(D7-Pad2)
- S8 pad 2: Net-(D8-Pad1) -> Net-(D8-Pad2)
- S9 pad 2: Net-(D9-Pad1) -> Net-(D9-Pad2)
Routing:
- net Net-(D38-Pad2): track 0.00 -> 84.3 mm
- net Net-(S37-Pad2): track 0.00 -> 72.4 mm
- net Net-(D26-Pad2): track 0.00 -> 50.3 mm
- net Net-(D25-Pad2): track 0.00 -> 46.2 mm
- net Net-(D13-Pad2): track 0.00 -> 27.0 mm
- net Net-(D14-Pad2): track 0.00 -> 26.8 mm
- net Net-(D2-Pad2): track 0.00 -> 6.10 mm
- net Net-(D1-Pad2): track 0.00 -> 6.10 mm

Commit message: 🚧 WIP - Place the components - Wire all the components
Parts:
- added REF**: MountingHole_3.5mm, ElsassKabel:MountingHole_3.5mm, F.Cu at (232.6, 125.4)
- added REF**: MountingHole_3.5mm, ElsassKabel:MountingHole_3.5mm, F.Cu at (50.4, 87.3)
- added REF**: Stabilizer_Cherry_MX_2.00u, ElsassKabel:Stabilizer_Cherry_MX_2.00u, F.Cu at (111.1, 134.9)
- added REF**: Stabilizer_Cherry_MX_2.00u, ElsassKabel:Stabilizer_Cherry_MX_2.00u, F.Cu at (125.4, 134.9)
- added REF**: MountingHole_3.5mm, ElsassKabel:MountingHole_3.5mm, F.Cu at (265.7, 48.3)
- added REF**: Stabilizer_Cherry_MX_7.00u, ElsassKabel:Stabilizer_Cherry_MX_7.00u, F.Cu at (146.8, 134.9)
- added REF**: MountingHole_3.5mm, ElsassKabel:MountingHole_3.5mm, F.Cu at (265.7, 63.3)
- added REF**: MountingHole_3.5mm, ElsassKabel:MountingHole_3.5mm, F.Cu at (32.8, 63.3)
- added REF**: MountingHole_3.5mm, ElsassKabel:MountingHole_3.5mm, F.Cu at (242.2, 87.3)
- added REF**: Stabilizer_Cherry_MX_2.00u, ElsassKabel:Stabilizer_Cherry_MX_2.00u, F.Cu at (165.9, 134.9)
- added REF**: MountingHole_3.5mm, ElsassKabel:MountingHole_3.5mm, F.Cu at (146.8, 87.3)
- added REF**: MountingHole_3.5mm, ElsassKabel:MountingHole_3.5mm, F.Cu at (59.8, 125.4)
- added REF**: MountingHole_3.5mm, ElsassKabel:MountingHole_3.5mm, F.Cu at (32.8, 48.3)
- added REF**: Stabilizer_Cherry_MX_6.25u, ElsassKabel:Stabilizer_Cherry_MX_6.25u, F.Cu at (154.0, 134.9)
- added REF**: Stabilizer_Cherry_MX_2.00u, ElsassKabel:Stabilizer_Cherry_MX_2.00u, F.Cu at (177.8, 134.9)
- added S53: SWITCH_2PIN, ElsassKabel:SW_Cherry_MX_PCB_6.25u, F.Cu at (154.0, 134.9)
- added S54: SWITCH_2PIN, ElsassKabel:SW_Cherry_MX_PCB_1.00u, F.Cu at (61.1, 134.9)
- added S55: SWITCH_2PIN, ElsassKabel:SW_Cherry_MX_PCB_1.25u, F.Cu at (82.5, 134.9)
- added S56: SWITCH_2PIN, ElsassKabel:SW_Cherry_MX_PCB_7.00u, F.Cu at (146.8, 134.9)
- added S57: SWITCH_2PIN, ElsassKabel:SW_Cherry_MX_PCB_1.00u, F.Cu at (37.3, 134.9)
- added S58: SWITCH_2PIN, ElsassKabel:SW_Cherry_MX_PCB_1.25u, F.Cu at (58.7, 134.9)
- added S59: SWITCH_2PIN, ElsassKabel:SW_Cherry_MX_PCB_1.00u, F.Cu at (80.2, 134.9)
- added S60: SWITCH_2PIN, ElsassKabel:SW_Cherry_MX_PCB_2.25u, F.Cu at (111.1, 134.9)
- added S61: SWITCH_2PIN, ElsassKabel:SW_Cherry_MX_PCB_1.00u, F.Cu at (142.1, 134.9)
- added S62: SWITCH_2PIN, ElsassKabel:SW_Cherry_MX_PCB_2.75u, F.Cu at (177.8, 134.9)
- S1, S10, S11, S14, S15, S16, S17, S18, S19, S2, S20, S21, S22, S23, S26, S27, S28, S29, S3, S30, S31, S32, S33, S34, S35, S36, S4, S45, S46, S47, S48, S5, S50, S51, S52, S6, S7, S8, S9: footprint Switch_Keyboard_Cherry_MX:SW_Cherry_MX_PCB_1.00u -> ElsassKabel:SW_Cherry_MX_PCB_1.00u
- S12, S25, S44: footprint Switch_Keyboard_Cherry_MX:SW_Cherry_MX_PCB_1.75u -> ElsassKabel:SW_Cherry_MX_PCB_1.75u
- S13, S37, S39, S42: footprint Switch_Keyboard_Cherry_MX:SW_Cherry_MX_PCB_1.25u -> ElsassKabel:SW_Cherry_MX_PCB_1.25u
- S24, S38, S43, S49: footprint Switch_Keyboard_Cherry_MX:SW_Cherry_MX_PCB_1.50u -> ElsassKabel:SW_Cherry_MX_PCB_1.50u
- S40: footprint Switch_Keyboard_Cherry_MX:SW_Cherry_MX_PCB_2.25u -> ElsassKabel:SW_Cherry_MX_PCB_2.25u
- S41: footprint Switch_Keyboard_Cherry_MX:SW_Cherry_MX_PCB_2.00u -> ElsassKabel:SW_Cherry_MX_PCB_2.00u
- USB1: value USB_C_GCT_USB4085 -> USB_C_Receptacle_USB2.0
- moved J1 232.8 mm to (114.3, 49.5), turned to 90 degrees
- moved C1 219.2 mm to (158.8, 53.0), turned to 90 degrees
- moved F1 213.1 mm to (139.7, 50.8), turned to 90 degrees
- moved USB1 211.5 mm to (149.2, 46.0)
- moved D51 206.5 mm to (157.5, 47.0), turned to 0 degrees
- moved SW1 204.7 mm to (90.7, 46.0)
- moved U1 204.1 mm to (175.3, 54.6)
- moved SW2 203.9 mm to (102.2, 46.0)
- moved C2 202.2 mm to (195.5, 44.5), turned to 180 degrees
- moved C4 196.8 mm to (189.2, 61.6)
- moved C5 196.8 mm to (204.5, 61.6)
- moved Y1 196.8 mm to (194.4, 60.3)
- moved R4 191.1 mm to (170.2, 58.4), turned to 180 degrees
- moved D49 190.5 mm to (156.8, 62.9), turned to 180 degrees
- moved D50 189.9 mm to (156.8, 59.7), turned to 180 degrees
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Connections:
- D1 pad 1: row0 -> MISO
- D10 pad 1: row0 -> MISO
- D11 pad 1: row0 -> MISO
- D12 pad 1: row0 -> MISO
- D13 pad 1: row1 -> MOSI
- D14 pad 1: row1 -> MOSI
- D15 pad 1: row1 -> MOSI
- D16 pad 1: row1 -> MOSI
- D17 pad 1: row1 -> MOSI
- D18 pad 1: row1 -> MOSI
- D19 pad 1: row1 -> MOSI
- D2 pad 1: row0 -> MISO
- D20 pad 1: row1 -> MOSI
- D21 pad 1: row1 -> MOSI
- D22 pad 1: row1 -> MOSI
- D23 pad 1: row1 -> MOSI
- D24 pad 1: row1 -> MOSI
- D3 pad 1: row0 -> MISO
- D37 pad 1: col1 -> row3
- D38 pad 1: col1 -> row3
- D39 pad 1: col1 -> row3
- D4 pad 1: row0 -> MISO
- D40 pad 1: col1 -> row3
- D41 pad 1: col1 -> row3
- D42 pad 1: col1 -> row3
- D42 pad 2: unconnected-(D42-Pad2) -> Net-(D42-Pad2)
- D43 pad 1: col1 -> row3
- D44 pad 1: col1 -> row3
- D44 pad 2: unconnected-(D44-Pad2) -> Net-(D44-Pad2)
- D45 pad 1: col1 -> row3
- D46 pad 1: col1 -> row3
- D47 pad 1: col1 -> row3
- D48 pad 1: col1 -> row3
- D5 pad 1: row0 -> MISO
- D6 pad 1: row0 -> MISO
- D7 pad 1: row0 -> MISO
- D8 pad 1: row0 -> MISO
- D9 pad 1: row0 -> MISO
- F1 pad 1: VCC -> +5V
- F1 pad 2: +5V -> VCC
- R1 pad 1: GND -> Net-(R1-Pad1)
- R1 pad 2: Net-(R1-Pad2) -> GND
- R2 pad 1: GND -> Net-(R2-Pad1)
- R2 pad 2: Net-(R2-Pad2) -> GND
- U1 pad 12: unconnected-(U1-Pad12) -> col9
- U1 pad 13: unconnected-(U1-Pad13) -> col10
- U1 pad 14: unconnected-(U1-Pad14) -> col11
- U1 pad 15: unconnected-(U1-Pad15) -> row3
- U1 pad 16: unconnected-(U1-Pad16) -> row2
- U1 pad 2: unconnected-(U1-Pad2) -> col3
- U1 pad 23: unconnected-(U1-Pad23) -> col7
- U1 pad 24: unconnected-(U1-Pad24) -> col6
- U1 pad 25: unconnected-(U1-Pad25) -> col4
- U1 pad 26: unconnected-(U1-Pad26) -> col2
- U1 pad 27: unconnected-(U1-Pad27) -> col1
- U1 pad 28: unconnected-(U1-Pad28) -> col0
- U1 pad 3: unconnected-(U1-Pad3) -> col5
- U1 pad 6: unconnected-(U1-Pad6) -> col8
- USB1 pad A1: (no net) -> GND
- USB1 pad A12: (no net) -> GND
- USB1 pad A4: (no net) -> VCC
- USB1 pad A5: (no net) -> Net-(R1-Pad1)
- USB1 pad A6: (no net) -> D+
- USB1 pad A7: (no net) -> D-
- USB1 pad A8: (no net) -> unconnected-(USB1-PadA8)
- USB1 pad A9: (no net) -> VCC
- USB1 pad B1: (no net) -> GND
- USB1 pad B12: (no net) -> GND
- USB1 pad B4: (no net) -> VCC
- USB1 pad B5: (no net) -> Net-(R2-Pad1)
- USB1 pad B6: (no net) -> D+
- USB1 pad B7: (no net) -> D-
- USB1 pad B8: (no net) -> unconnected-(USB1-PadB8)
- USB1 pad B9: (no net) -> VCC
- USB1 pad S1: (no net) -> GND
Routing:
- net MISO: track 0.00 -> 391.1 mm, vias 0 -> 5
- net MOSI: track 0.00 -> 385.3 mm, vias 0 -> 4
- net row2: track 0.00 -> 281.7 mm, vias 0 -> 3
- net row3: track 0.00 -> 268.0 mm, vias 0 -> 3
- net col0: track 0.00 -> 232.3 mm
- net col1: track 0.00 -> 225.8 mm
- net col2: track 0.00 -> 204.5 mm
- net col3: track 0.00 -> 176.7 mm
- net col4: track 0.00 -> 174.6 mm
- net +5V: track 0.00 -> 170.9 mm
- net col5: track 0.00 -> 142.7 mm
- net col11: track 0.00 -> 127.5 mm
- net col6: track 0.00 -> 122.5 mm
- net Net-(D44-Pad2): track 0.00 -> 119.2 mm
- net BOOT: track 0.00 -> 117.7 mm, vias 0 -> 2
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- added copper zone on B.Cu, net GND
- added copper zone on F.Cu, net GND
Other:
- board outline added: 242.9 x 101.2 mm
